File: hardware/pcb/devkit-carrier-v1/sesame-devkit-carrier.kicad_sch (KiCad schematic)
At the start: 28 parts, among them J1 DevKit L, J2 DevKit R, J3 OLED, J4 IO, J5 IO2, J6 Battery pigtail, SW1 Switch, U1 Pololu D24V50F5

Commit message: Carrier PCB: wider short-risk margins and a short_check.py gate
Ground fill 0.5 mm back from all copper (was 0.3), C3 on 2.5 mm pitch
with narrowed pads (1.3 mm gap across the battery), R1/R2 battery-to-GND
pads 2.2 mm apart, stitching vias moved off the 5V feed. short_check.py
(plain Python, no KiCad) enforces the margins. ERC/DRC/parity/audit clean,
kicad-happy unchanged.

Co-Authored-By: Claude Opus 5.5 <noreply@anthropic.com>
Parts:
- C3: footprint Sesame:CP_Radial_D5.0mm_P2.00mm -> Sesame:CP_Radial_D5.0mm_P2.50mm
Changed lines of the file:
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@@
 	(wire (pts (xy 190.50 128.27) (xy 190.50 133.35)) (stroke (width 0) (type default)))
 	(symbol (lib_id "power:GND") (at 190.50 133.35 0) (unit 1) (exclude_from_sim no) (in_bom no) (on_board no) (dnp no) (property "Reference" "#PWR03" (at 190.50 128.27 0) (effects (font (size 1.27 1.27)) (hide yes))) (property "Value" "GND" (at 190.50 139.35 0) (effects (font (size 1.27 1.27)))) (property "Footprint" "" (at 190.50 133.35 0) (effects (font (size 1.27 1.27)) (hide yes))) (property "Datasheet" "" (at 190.50 133.35 0) (effects (font (size 1.27 1.27)) (hide yes))) (property "Description" "" (at 190.50 133.35 0) (effects (font (size 1.27 1.27)) (hide yes))) (pin "1") (instances (project "sesame-devkit-carrier" (path "/38fbc7a5-229d-5e0a-bd26-42fc2efc63f6" (reference "#PWR03") (unit 1)))))
-	(symbol (lib_id "Device:C_Polarized") (at 373.38 109.22 0) (unit 1) (exclude_from_sim no) (in_bom yes) (on_board yes) (dnp no) (property "Reference" "C3" (at 373.38 104.14 0) (effects (font (size 1.27 1.27)))) (property "Value" "47uF 35V" (at 373.38 105.92 0) (effects (font (size 1.27 1.27)))) (property "Footprint" "Sesame:CP_Radial_D5.0mm_P2.00mm" (at 373.38 109.22 0) (effects (font (size 1.27 1.27)) (hide yes))) (property "Datasheet" "" (at 373.38 109.22 0) (effects (font (size 1.27 1.27)) (hide yes))) (property "Description" "" (at 373.38 109.22 0) (effects (font (size 1.27 1.27)) (hide yes))) (pin "1")(pin "2") (instances (project "sesame-devkit-carrier" (path "/38fbc7a5-229d-5e0a-bd26-42fc2efc63f6" (reference "C3") (unit 1)))))
+	(symbol (lib_id "Device:C_Polarized") (at 373.38 109.22 0) (unit 1) (exclude_from_sim no) (in_bom yes) (on_board yes) (dnp no) (property "Reference" "C3" (at 373.38 104.14 0) (effects (font (size 1.27 1.27)))) (property "Value" "47uF 35V" (at 373.38 105.92 0) (effects (font (size 1.27 1.27)))) (property "Footprint" "Sesame:CP_Radial_D5.0mm_P2.50mm" (at 373.38 109.22 0) (effects (font (size 1.27 1.27)) (hide yes))) (property "Datasheet" "" (at 373.38 109.22 0) (effects (font (size 1.27 1.27)) (hide yes))) (property "Description" "" (at 373.38 109.22 0) (effects (font (size 1.27 1.27)) (hide yes))) (pin "1")(pin "2") (instances (project "sesame-devkit-carrier" (path "/38fbc7a5-229d-5e0a-bd26-42fc2efc63f6" (reference "C3") (unit 1)))))
 	(wire (pts (xy 373.38 105.41) (xy 373.38 100.33)) (stroke (width 0) (type default)))
 	(global_label "VBAT_SW" (shape passive) (at 373.38 100.33 90) (fields_autoplaced yes) (effects (font (size 1.27 1.27)) (justify left)) (property "Intersheetrefs" "${INTERSHEET_REFS}" (at 373.38 100.33 0) (effects (font (size 1.27 1.27)) (justify left) (hide yes))))
